File: matrix.kicad_sch (KiCad schematic)
At the start: 134 parts

Commit message: Update 3d models
Parts:
- D1, D10, D11, D12, D13, D14, D15, D16, D17, D18, D19, D2, D20, D21, D22, D23, D24, D25, D26, D27, D28, D29, D3, D30, D31, D32, D33, D34, D35, D36, D37, D38, D39, D4, D40, D41, D42, D43, D44, D45, D46, D47, D48, D49, D5, D50, D51, D52, D53, D54, D55, D56, D57, D58, D59, D6, D60, D61, D62, D63, D64, D65, D66, D67, D7, D8, D9: value (none) -> D; footprint (none) -> Diodes_SMD:D_SOD-123
- SW1, SW10, SW11, SW12, SW13, SW15, SW16, SW17, SW18, SW19, SW20, SW21, SW22, SW24, SW25, SW26, SW27, SW28, SW29, SW30, SW31, SW32, SW33, SW34, SW35, SW36, SW38, SW39, SW40, SW41, SW42, SW43, SW44, SW45, SW47, SW48, SW49, SW50, SW51, SW52, SW53, SW55, SW56, SW58, SW59, SW6, SW61, SW62, SW63, SW64, SW65, SW66, SW67, SW7, SW8, SW9: value (none) -> SW_Push; footprint (none) -> MX_Switch:SW_Cherry_MX_1.00u_PCB
- SW14, SW2, SW46, SW5, SW60: value (none) -> SW_Push; footprint (none) -> MX_Switch:SW_Cherry_MX_1.50u_PCB
- SW23: value (none) -> SW_Push; footprint (none) -> MX_Switch:SW_Cherry_MX_2.00u_PCB_ReversedStabilizers
- SW3, SW54: value (none) -> SW_Push; footprint (none) -> MX_Switch:SW_Cherry_MX_1.75u_PCB
- SW37: value (none) -> SW_Push; footprint (none) -> MX_Switch:SW_Cherry_MX_2.75u_PCB_ReversedStabilizers
- SW4: value (none) -> SW_Push; footprint (none) -> MX_Switch:SW_Cherry_MX_2.25u_PCB
- SW57: value (none) -> SW_Push; footprint (none) -> MX_Switch:SW_Cherry_MX_2.25u_PCB_ReversedStabilizers

Commit message: new layout
Parts:
- removed D54, D58, D61, D62, D64, D65: D, Diodes_SMD:D_SOD-123, symbol Device:D
- removed SW54: SW_Push, MX_Switch:SW_Cherry_MX_1.75u_PCB, symbol Switch:SW_Push
- removed SW58, SW61, SW62, SW64, SW65: SW_Push, MX_Switch:SW_Cherry_MX_1.00u_PCB, symbol Switch:SW_Push
- added D1, D2, D3, D55, D60, D8: D, Diodes_SMD:D_SOD-123, symbol Device:D
- added SW1, SW2, SW3: SW_Push, MX_Switch:SW_Cherry_MX_1.00u_PCB, symbol Switch:SW_Push
- added SW55, SW60, SW8: SW_Push, MX_Switch:SW_Cherry_MX_1.50u_PCB, symbol Switch:SW_Push
- SW59: footprint MX_Switch:SW_Cherry_MX_1.00u_PCB -> MX_Switch:SW_Cherry_MX_2.00u_PCB_ReversedStabilizers
- SW63: footprint MX_Switch:SW_Cherry_MX_1.00u_PCB -> MX_Switch:SW_Cherry_MX_2.00u_PCB
- renumbered D7 to D10, D8 to D11, D9 to D12, D5 to D13, D10 to D14, D11 to D15, D12 to D16, D13 to D17, D14 to D18, D15 to D19, D16 to D20, D17 to D21, D18 to D22, D19 to D23, D20 to D24, D21 to D25, D22 to D26, D23 to D27, D24 to D28, D25 to D29, D26 to D30, D27 to D31, D28 to D32, D29 to D33, D30 to D34, D31 to D35, D32 to D36, D33 to D38, D34 to D39, D1 to D4, D35 to D40, D36 to D41, D38 to D42, D39 to D43, D40 to D44, D41 to D45, D42 to D47, D43 to D48, D44 to D49, D2 to D5, D45 to D50, D47 to D51, D48 to D52, D49 to D53, D50 to D54, D51 to D56, D52 to D57, D53 to D58, D3 to D6, D55 to D61, D56 to D62, D60 to D64, D57 to D65, D4 to D7, D6 to D9, SW7 to SW10, SW8 to SW11, SW9 to SW12, SW5 to SW13, SW10 to SW14, SW11 to SW15, SW12 to SW16, SW13 to SW17, SW14 to SW18, SW15 to SW19, SW16 to SW20, SW17 to SW21, SW18 to SW22, SW19 to SW23, SW20 to SW24, SW21 to SW25, SW22 to SW26, SW23 to SW27, SW24 to SW28, SW25 to SW29, SW26 to SW30, SW27 to SW31, SW28 to SW32, SW29 to SW33, SW30 to SW34, SW31 to SW35, SW32 to SW36, SW33 to SW38, SW34 to SW39, SW1 to SW4, SW35 to SW40, SW36 to SW41, SW38 to SW42, SW39 to SW43, SW40 to SW44, SW41 to SW45, SW42 to SW47, SW43 to SW48, SW44 to SW49, SW2 to SW5, SW45 to SW50, SW47 to SW51, SW48 to SW52, SW49 to SW53, SW50 to SW54, SW51 to SW56, SW52 to SW57, SW53 to SW58, SW3 to SW6, SW55 to SW61, SW56 to SW62, SW60 to SW64, SW57 to SW65, SW4 to SW7, SW6 to SW9
Connections:
- net col14 is gone; now on net col13: SW63.1, SW66.1, SW67.1
- net col0: now also SW8.1; no longer SW13.1
- net col1: now also SW13.1
- net col10: now also SW55.1
- net col11: now also SW59.1, SW60.1
- net col12: no longer SW65.1
- net col13: now also SW65.1; no longer SW59.1
- net col6: no longer SW34.1, SW35.1, SW36.1
- net col7: no longer SW37.1
- net col8: now also SW46.1
- net col9: no longer SW46.1
- net row0: no longer D38.1 (K), D42.1 (K), D47.1 (K), D51.1 (K), D56.1 (K), D59.1 (K), D61.1 (K), D63.1 (K)
- net row1: no longer D34.1 (K), D39.1 (K), D43.1 (K), D48.1 (K), D52.1 (K), D57.1 (K), D62.1 (K), D64.1 (K)
- net row2: no longer D35.1 (K), D40.1 (K), D44.1 (K), D49.1 (K), D53.1 (K), D58.1 (K), D65.1 (K)
- net row3: no longer D36.1 (K), D41.1 (K), D45.1 (K), D50.1 (K), D54.1 (K), D66.1 (K)
- net row4: now also D8.1 (K); no longer D37.1 (K), D46.1 (K), D67.1 (K)
- new net: SW34.1, SW35.1, SW36.1, SW37.1
- new net: D34.1 (K), D39.1 (K), D43.1 (K), D48.1 (K), D52.1 (K), D57.1 (K), D62.1 (K), D64.1 (K)
- new net: D35.1 (K), D40.1 (K), D44.1 (K), D49.1 (K), D53.1 (K), D58.1 (K), D65.1 (K)
- new net: D36.1 (K), D41.1 (K), D45.1 (K), D50.1 (K), D54.1 (K), D59.1 (K), D66.1 (K)
- new net: D38.1 (K), D42.1 (K), D47.1 (K), D51.1 (K), D56.1 (K), D61.1 (K)
- new net: D37.1 (K), D46.1 (K), D55.1 (K), D60.1 (K), D67.1 (K)
- new net: D60.2 (A), SW60.2
- new net: D1.2 (A), SW1.2
- new net: D8.2 (A), SW8.2
- new net: SW1.1, SW2.1, SW3.1
- new net: D3.2 (A), SW3.2
- new net: D2.2 (A), SW2.2
- new net: D55.2 (A), SW55.2
Other:
- note removed: "DOWN"
- note removed: "LEFT"
- note removed: "M1"
- note removed: "M2"
- note removed: "M3"
- note removed: "RGHT"
- note removed: "UP"
- note removed: "`"
- note removed: "|"
- moved on the sheet: D13, D34, D35, D36, D37, D38, D39, D40, D41, D42, D43, D44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

Commit message: scripting tests
Parts:
- D1, D10, D11, D12, D13, D14, D15, D16, D17, D18, D19, D2, D20, D21, D22, D23, D24, D25, D26, D27, D28, D29, D3, D30, D31, D32, D33, D34, D35, D36, D37, D38, D39, D4, D40, D41, D42, D43, D44, D45, D46, D47, D48, D49, D5, D50, D51, D52, D53, D54, D55, D56, D57, D58, D59, D6, D60, D61, D62, D63, D64, D65, D66, D67, D7, D8, D9: footprint Diodes_SMD:D_SOD-123 -> Diode_SMD:D_SOD-123
