File: arisu.kicad_pcb (KiCad board)
At the start: 2 copper layers, 343 x 119 mm, 166 parts, among them J1 Conn_01x02, J2 USB_B_Micro, SW1 SW_Push, SW10 SW_Push, SW11 SW_Push, SW12 SW_Push, SW13 SW_Push, SW14 SW_Push, SW15 SW_Push, SW16 SW_Push, SW17 SW_Push, SW18 SW_Push, SW19 SW_Push, SW2 SW_Push, SW20 SW_Push, SW21 SW_Push, SW22 SW_Push, SW23 SW_Push, SW24 SW_Push, SW25 SW_Push, SW26 SW_Push, SW27 SW_Push, SW28 SW_Push, SW29 SW_Push, SW3 SW_Push, SW30 SW_Push, SW31 SW_Push, SW32 SW_Push, SW33 SW_Push, SW34 SW_Push, SW35 SW_Push, SW36 SW_Push, SW37 SW_Push, SW38 SW_Push, SW39 SW_Push, SW4 SW_Push, SW40 SW_Push, SW41 SW_Push, SW42 SW_Push, SW43 SW_Push, SW44 SW_Push, SW45 SW_Push, SW46 SW_Push, SW47 SW_Push, SW48 SW_Push, SW49 SW_Push, SW5 SW_Push, SW50 SW_Push, SW51 SW_Push, SW52 SW_Push, SW53 SW_Push, SW54 SW_Push, SW55 SW_Push, SW56 SW_Push, SW57 SW_Push, SW58 SW_Push, SW59 SW_Push, SW6 SW_Push, SW60 SW_Push, SW61 SW_Push, SW62 SW_Push, SW63 SW_Push, SW64 SW_Push, SW65 SW_Push, SW66 SW_Push, SW67 SW_Push, SW7 SW_Push, SW8 SW_Push, SW9 SW_Push, U1 W25Q128JVS, U2 NCP1117-3.3_SOT223, U3 RP2040, Y1 ABLS-12.000MHZ-B4-T

Commit message: Split the keyboard into multiple files, give both sides a micro, and added 1 of the 2 jack circuits
Parts:
- added C17: 27p, Capacitor_SMD:C_0402_1005Metric, F.Cu at (109.3, 163.4)
- added C18: 27p, Capacitor_SMD:C_0402_1005Metric, F.Cu at (114.0, 160.1)
- added C19: 10u, Capacitor_SMD:C_0805_2012Metric, F.Cu at (94.1, 174.3)
- added C20: 100n, Capacitor_SMD:C_0402_1005Metric, F.Cu at (94.2, 162.4)
- added C21: 10u, Capacitor_SMD:C_0805_2012Metric, F.Cu at (104.3, 165.0)
- added C22: 100n, Capacitor_SMD:C_0402_1005Metric, F.Cu at (114.0, 158.2)
- added C23: 100n, Capacitor_SMD:C_0402_1005Metric, F.Cu at (110.9, 165.4)
- added C24: 1u, Capacitor_SMD:C_0402_1005Metric, F.Cu at (106.4, 169.4)
- added C25: 100n, Capacitor_SMD:C_0402_1005Metric, F.Cu at (106.4, 167.5)
- added C26: 1u, Capacitor_SMD:C_0402_1005Metric, F.Cu at (112.2, 163.4)
- added C27: 100n, Capacitor_SMD:C_0402_1005Metric, F.Cu at (103.5, 169.4)
- added C28: 100n, Capacitor_SMD:C_0402_1005Metric, F.Cu at (116.9, 160.1)
- added C29: 100n, Capacitor_SMD:C_0402_1005Metric, F.Cu at (116.9, 158.2)
- added C30: 100n, Capacitor_SMD:C_0402_1005Metric, F.Cu at (116.9, 156.2)
- added C31: 100n, Capacitor_SMD:C_0402_1005Metric, F.Cu at (97.8, 173.7)
- added C32: 100n, Capacitor_SMD:C_0402_1005Metric, F.Cu at (97.8, 175.7)
- added J3: USB_B_Micro, RP2040_minimal:USB_Micro-B_Amphenol_10103594-0001LF_Horizontal_modified, F.Cu at (87.2, 173.2)
- added J4: Conn_01x02, Connector_PinHeader_2.54mm:PinHeader_1x02_P2.54mm_Vertical, F.Cu at (110.2, 157.5)
- added R10: 27, Capacitor_SMD:C_0402_1005Metric, F.Cu at (100.6, 173.7)
- added R6: 1k, Capacitor_SMD:C_0402_1005Metric, F.Cu at (108.0, 165.4)
- added R7: DNF, Capacitor_SMD:C_0402_1005Metric, F.Cu at (103.5, 167.5)
- added R8: 1k, Capacitor_SMD:C_0402_1005Metric, F.Cu at (103.5, 171.4)
- added R9: 27, Capacitor_SMD:C_0402_1005Metric, F.Cu at (114.0, 156.2)
- added U4: NCP1117-3.3_SOT223, Package_TO_SOT_SMD:SOT-223-3_TabPin2, F.Cu at (103.0, 159.3)
- added U5: W25Q128JVS, Package_SO:SOIC-8_5.23x5.23mm_P1.27mm, F.Cu at (87.6, 164.8)
- added U6: RP2040, RP2040_minimal:RP2040-QFN-56, F.Cu at (97.5, 168.1)
- added Y2: ABLS-12.000MHZ-B4-T, RP2040_minimal:Crystal_SMD_HC49-US, F.Cu at (90.3, 158.3)
- J1: value Conn_01x02 -> USB_B_Micro; footprint Connector_PinHeader_2.54mm:PinHeader_1x02_P2.54mm_Vertical -> RP2040_minimal:USB_Micro-B_Amphenol_10103594-0001LF_Horizontal_modified
- J2: value USB_B_Micro -> Conn_01x02; footprint RP2040_minimal:USB_Micro-B_Amphenol_10103594-0001LF_Horizontal_modified -> Connector_PinHeader_2.54mm:PinHeader_1x02_P2.54mm_Vertical
- U1: value W25Q128JVS -> NCP1117-3.3_SOT223; footprint Package_SO:SOIC-8_5.23x5.23mm_P1.27mm -> Package_TO_SOT_SMD:SOT-223-3_TabPin2
- U2: value NCP1117-3.3_SOT223 -> W25Q128JVS; footprint Package_TO_SOT_SMD:SOT-223-3_TabPin2 -> Package_SO:SOIC-8_5.23x5.23mm_P1.27mm
- moved C10 213.5 mm to (281.2, 162.8)
- moved C11 213.5 mm to (275.4, 170.8)
- moved C12 213.5 mm to (279.8, 164.8)
- moved C13 213.5 mm to (285.8, 155.6)
- moved C14 213.5 mm to (266.1, 161.8)
- moved C16 213.5 mm to (278.2, 166.9)
- moved C2 213.5 mm to (282.7, 164.8)
- moved C4 213.5 mm to (285.8, 159.5)
- moved C5 213.5 mm to (265.9, 173.7)
- moved C6 213.5 mm to (285.8, 157.6)
- moved C7 213.5 mm to (275.4, 166.9)
- moved J1 213.5 mm to (282.1, 156.9)
- moved J2 213.5 mm to (259.0, 172.6)
- moved R1 213.5 mm to (278.2, 168.8)
- moved R2 213.5 mm to (275.4, 168.8)
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Connections:
- net /RUN renamed /Right/RUN
- net /SWCLK renamed /Right/SWCLK
- net /SWD renamed /Right/SWD
- net /XIN renamed /Right/XIN
- net /XOUT renamed /Right/XOUT
- net /col0 renamed /Left/col1L
- net /col1 renamed /Left/col2L
- net /col13 renamed /Right/matrixR/col7
- net /col2 renamed /Left/col3L
- net /col4 renamed /Left/col5L
- net /col5 renamed /Left/col6L
- net /row3 renamed /Left/row3L
- net Net-(SW1-Pad1) renamed /Left/col0L
- D1 pad 1: unconnected-(D1-Pad1) -> /Left/row0L
- D10 pad 1: /row1 -> /Left/row1L
- D11 pad 1: /row2 -> /Left/row2L
- D13 pad 1: /row4 -> /Left/row4L
- D14 pad 1: /row0 -> /Left/row0L
- D15 pad 1: /row1 -> /Left/row1L
- D16 pad 1: /row2 -> /Left/row2L
- D18 pad 1: /row4 -> /Left/row4L
- D19 pad 1: /row0 -> /Left/row0L
- D2 pad 1: unconnected-(D2-Pad1) -> /Left/row1L
- D20 pad 1: /row1 -> /Left/row1L
- D21 pad 1: /row2 -> /Left/row2L
- D23 pad 1: /row0 -> /Left/row0L
- D24 pad 1: /row1 -> /Left/row1L
- D25 pad 1: /row2 -> /Left/row2L
- D27 pad 1: /row4 -> /Left/row4L
- D28 pad 1: /row0 -> /Left/row0L
- D29 pad 1: /row1 -> /Left/row1L
- D3 pad 1: unconnected-(D3-Pad1) -> /Left/row2L
- D30 pad 1: /row2 -> /Left/row2L
- D32 pad 1: /row4 -> /Left/row4L
- D33 pad 1: /row0 -> /Left/row4L
- D34 pad 1: Net-(D34-Pad1) -> /Right/row1L
- D35 pad 1: Net-(D35-Pad1) -> /Right/row2L
- D36 pad 1: Net-(D36-Pad1) -> /Right/row3L
- D37 pad 1: Net-(D37-Pad1) -> /Right/row4L
- D38 pad 1: Net-(D38-Pad1) -> /Right/row0L
- D39 pad 1: Net-(D34-Pad1) -> /Right/row1L
- D4 pad 1: /row0 -> /Left/row0L
- D40 pad 1: Net-(D35-Pad1) -> /Right/row2L
- D41 pad 1: Net-(D36-Pad1) -> /Right/row3L
- D42 pad 1: Net-(D38-Pad1) -> /Right/row0L
- D43 pad 1: Net-(D34-Pad1) -> /Right/row1L
- D44 pad 1: Net-(D35-Pad1) -> /Right/row2L
- D45 pad 1: Net-(D36-Pad1) -> /Right/row3L
- D46 pad 1: Net-(D37-Pad1) -> /Right/row4L
- D47 pad 1: Net-(D38-Pad1) -> /Right/row0L
- D48 pad 1: Net-(D34-Pad1) -> /Right/row1L
- D49 pad 1: Net-(D35-Pad1) -> /Right/row2L
- D5 pad 1: /row1 -> /Left/row1L
- D50 pad 1: Net-(D36-Pad1) -> /Right/row3L
- D51 pad 1: Net-(D38-Pad1) -> /Right/row0L
- D52 pad 1: Net-(D34-Pad1) -> /Right/row1L
- D53 pad 1: Net-(D35-Pad1) -> /Right/row2L
- D54 pad 1: Net-(D36-Pad1) -> /Right/row3L
- D55 pad 1: Net-(D37-Pad1) -> /Right/row4L
- D56 pad 1: Net-(D38-Pad1) -> /Right/row0L
- D57 pad 1: Net-(D34-Pad1) -> /Right/row1L
- D58 pad 1: Net-(D35-Pad1) -> /Right/row2L
- D59 pad 1: Net-(D36-Pad1) -> /Right/row3L
- D6 pad 1: /row2 -> /Left/row2L
- D60 pad 1: Net-(D37-Pad1) -> /Right/row4L
- D61 pad 1: Net-(D38-Pad1) -> /Right/row0L
- D62 pad 1: Net-(D34-Pad1) -> /Right/row1L
- D63 pad 1: unconnected-(D63-Pad1) -> /Right/row0L
- D64 pad 1: Net-(D34-Pad1) -> /Right/row1L
- D65 pad 1: Net-(D35-Pad1) -> /Right/row2L
- D66 pad 1: Net-(D36-Pad1) -> /Right/row3L
- D67 pad 1: Net-(D37-Pad1) -> /Right/row4L
- D8 pad 1: /row4 -> /Left/row4L
- D9 pad 1: /row0 -> /Left/row0L
- J1 pad 1: /~{USB_BOOT} -> VBUS
- J1 pad 2: GND -> /Right/USB_D-
- J2 pad 1: VBUS -> /Right/~{USB_BOOT}
- J2 pad 2: /USB_D- -> GND
- R1 pad 1: /QSPI_SS -> /Right/QSPI_SS
- R1 pad 2: /~{USB_BOOT} -> /Right/~{USB_BOOT}
- R2 pad 2: /QSPI_SS -> /Right/QSPI_SS
- R4 pad 1: /USB_D+ -> /Right/USB_D+
- R5 pad 1: /USB_D- -> /Right/USB_D-
- SW19 pad 1: /col3 -> /Left/col4L
- SW20 pad 1: /col3 -> /Left/col4L
- SW21 pad 1: /col3 -> /Left/col4L
- SW22 pad 1: /col3 -> /Left/col4L
- SW33 pad 1: /col6 -> /Left/col4L
- SW34 pad 1: Net-(SW34-Pad1) -> /Right/col0L
- SW35 pad 1: Net-(SW34-Pad1) -> /Right/col0L
- SW36 pad 1: Net-(SW34-Pad1) -> /Right/col0L
- SW37 pad 1: Net-(SW34-Pad1) -> /Right/col0L
- SW38 pad 1: /col7 -> /Right/col1L
- SW39 pad 1: /col7 -> /Right/col1L
- SW40 pad 1: /col7 -> /Right/col1L
- SW41 pad 1: /col7 -> /Right/col1L
- SW42 pad 1: /col8 -> /Right/col2L
- SW43 pad 1: /col8 -> /Right/col2L
- SW44 pad 1: /col8 -> /Right/col2L
- SW45 pad 1: /col8 -> /Right/col2L
- SW46 pad 1: /col8 -> /Right/col2L
- SW47 pad 1: /col9 -> /Right/col3L
- SW48 pad 1: /col9 -> /Right/col3L
- SW49 pad 1: /col9 -> /Right/col3L
- SW50 pad 1: /col9 -> /Right/col3L
- SW51 pad 1: /col10 -> /Right/col4L
- SW52 pad 1: /col10 -> /Right/col4L
- SW53 pad 1: /col10 -> /Right/col4L
- SW54 pad 1: /col10 -> /Right/col4L
- SW55 pad 1: /col10 -> /Right/col4L
- SW56 pad 1: /col11 -> /Right/col5L
- SW57 pad 1: /col11 -> /Right/col5L
- SW58 pad 1: /col11 -> /Right/col5L
- SW59 pad 1: /col11 -> /Right/col5L
- SW60 pad 1: /col11 -> /Right/col5L
- SW61 pad 1: /col12 -> /Right/col6L
- SW62 pad 1: /col12 -> /Right/col6L
- U1 pad 1: /QSPI_SS -> GND
- U1 pad 2: /QSPI_SD1 -> +3V3
- U1 pad 3: /QSPI_SD2 -> VBUS
- U2 pad 1: GND -> /Right/QSPI_SS
- U2 pad 2: +3V3 -> /Right/QSPI_SD1
- U2 pad 3: VBUS -> /Right/QSPI_SD2
- U3 pad 11: /GPIO8 -> /Right/row0L
- U3 pad 12: /GPIO9 -> /Right/row1L
- U3 pad 13: /GPIO10 -> /Right/row2L
- U3 pad 14: /GPIO11 -> /Right/row3L
- U3 pad 15: /GPIO12 -> /Right/row4L
- U3 pad 16: /GPIO13 -> unconnected-(U3-Pad16)
- U3 pad 17: /GPIO14 -> unconnected-(U3-Pad17)
- U3 pad 18: /GPIO15 -> unconnected-(U3-Pad18)
- U3 pad 2: /GPIO0 -> /Right/col0L
- U3 pad 27: /GPIO16 -> unconnected-(U3-Pad27)
- U3 pad 28: /GPIO17 -> unconnected-(U3-Pad28)
- U3 pad 29: /GPIO18 -> unconnected-(U3-Pad29)
- U3 pad 3: /GPIO1 -> /Right/col1L
- U3 pad 30: /GPIO19 -> unconnected-(U3-Pad30)
- U3 pad 31: /GPIO20 -> unconnected-(U3-Pad31)
- U3 pad 32: /GPIO21 -> unconnected-(U3-Pad32)
- U3 pad 34: /GPIO22 -> unconnected-(U3-Pad34)
- U3 pad 35: /GPIO23 -> unconnected-(U3-Pad35)
- U3 pad 36: /GPIO24 -> unconnected-(U3-Pad36)
- U3 pad 37: /GPIO25 -> unconnected-(U3-Pad37)
- U3 pad 38: /GPIO26_ADC0 -> unconnected-(U3-Pad38)
- U3 pad 39: /GPIO27_ADC1 -> unconnected-(U3-Pad39)
- U3 pad 4: /GPIO2 -> /Right/col2L
- U3 pad 40: /GPIO28_ADC2 -> unconnected-(U3-Pad40)
- U3 pad 41: /GPIO29_ADC3 -> unconnected-(U3-Pad41)
- U3 pad 5: /GPIO3 -> /Right/col3L
- U3 pad 51: /QSPI_SD3 -> /Right/QSPI_SD3
- U3 pad 52: /QSPI_SCLK -> /Right/QSPI_SCLK
- U3 pad 53: /QSPI_SD0 -> /Right/QSPI_SD0
- U3 pad 54: /QSPI_SD2 -> /Right/QSPI_SD2
- U3 pad 55: /QSPI_SD1 -> /Right/QSPI_SD1
- U3 pad 56: /QSPI_SS -> /Right/QSPI_SS
- U3 pad 6: /GPIO4 -> /Right/col4L
- U3 pad 7: /GPIO5 -> /Right/col5L
- U3 pad 8: /GPIO6 -> /Right/col6L
- U3 pad 9: /GPIO7 -> unconnected-(U3-Pad9)
Routing:
- net /col11: track 97.0 -> 0.00 mm
- net /Right/col5L: track 0.00 -> 97.0 mm
- net /col10: track 90.1 -> 0.00 mm
- net /Right/col4L: track 0.00 -> 90.1 mm
- net /col8: track 86.7 -> 0.00 mm
- net /Right/col2L: track 0.00 -> 86.7 mm
- net /col3: track 65.6 -> 0.00 mm
- net /Left/col4L: track 0.00 -> 65.6 mm
- net /col7: track 64.6 -> 0.00 mm
- net /Right/col1L: track 0.00 -> 64.6 mm
- net /col9: track 64.6 -> 0.00 mm
- net /Right/col3L: track 0.00 -> 64.6 mm
- net Net-(SW34-Pad1): track 64.1 -> 0.00 mm
- net /Right/col0L: track 0.00 -> 64.1 mm
- net /col12: track 24.7 -> 0.00 mm
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
Commit message: No more erc errors + centering and socketing of switches
Parts:
- removed C17, C18: 27p, Capacitor_SMD:C_0402_1005Metric
- removed C19, C21: 10u, Capacitor_SMD:C_0805_2012Metric
- removed C20, C22, C23, C25, C27, C28, C29, C30, C31, C32: 100n, Capacitor_SMD:C_0402_1005Metric
- removed C24, C26: 1u, Capacitor_SMD:C_0402_1005Metric
- removed J1, J3: USB_B_Micro, RP2040_minimal:USB_Micro-B_Amphenol_10103594-0001LF_Horizontal_modified
- removed J4: Conn_01x02, Connector_PinHeader_2.54mm:PinHeader_1x02_P2.54mm_Vertical
- removed R10, R9: 27, Capacitor_SMD:C_0402_1005Metric
- removed R6, R8: 1k, Capacitor_SMD:C_0402_1005Metric
- removed R7: DNF, Capacitor_SMD:C_0402_1005Metric
- removed U4: NCP1117-3.3_SOT223, Package_TO_SOT_SMD:SOT-223-3_TabPin2
- removed U5: W25Q128JVS, Package_SO:SOIC-8_5.23x5.23mm_P1.27mm
- removed U6: RP2040, RP2040_minimal:RP2040-QFN-56
- removed Y2: ABLS-12.000MHZ-B4-T, RP2040_minimal:Crystal_SMD_HC49-US
- SW1, SW10, SW11, SW12, SW14, SW15, SW16, SW17, SW19, SW2, SW20, SW21, SW22, SW23, SW24, SW25, SW26, SW28, SW29, SW3, SW30, SW31, SW32, SW33, SW34, SW35, SW36, SW38, SW39, SW4, SW40, SW41, SW42, SW43, SW44, SW45, SW47, SW48, SW49, SW50, SW51, SW52, SW53, SW54, SW56, SW57, SW58, SW61, SW62, SW66, SW67, SW9: footprint MX_Switch:SW_Cherry_MX_1.00u_PCB -> MX_Switch:SW_Cherry_MX_1.00u_PCB_Socket
- SW13, SW18, SW46, SW5, SW55, SW60, SW64, SW8: footprint MX_Switch:SW_Cherry_MX_1.50u_PCB -> MX_Switch:SW_Cherry_MX_1.50u_PCB_Socket
- SW27, SW59: footprint MX_Switch:SW_Cherry_MX_2.00u_PCB_ReversedStabilizers -> MX_Switch:SW_Cherry_MX_2.00u_PCB_Socket_ReversedStabilizers
- SW37: footprint MX_Switch:SW_Cherry_MX_2.75u_PCB_ReversedStabilizers -> MX_Switch:SW_Cherry_MX_2.75u_PCB_Socket_ReversedStabilizers
- SW6: footprint MX_Switch:SW_Cherry_MX_1.75u_PCB -> MX_Switch:SW_Cherry_MX_1.75u_PCB_Socket
- SW63: footprint MX_Switch:SW_Cherry_MX_2.00u_PCB -> MX_Switch:SW_Cherry_MX_2.00u_PCB_Socket
- SW65: footprint MX_Switch:SW_Cherry_MX_2.25u_PCB_ReversedStabilizers -> MX_Switch:SW_Cherry_MX_2.25u_PCB_Socket_ReversedStabilizers
- SW7: footprint MX_Switch:SW_Cherry_MX_2.25u_PCB -> MX_Switch:SW_Cherry_MX_2.25u_PCB_Socket_ReversedStabilizers
- moved R3 44.4 mm to (244.9, 163.0)
- moved C4 41.7 mm to (244.9, 167.5)
- moved C13 38.8 mm to (247.8, 163.0)
- moved C3 35.0 mm to (241.2, 166.6)
- moved C12 34.9 mm to (244.9, 165.0)
- moved U2 30.6 mm to (244.2, 158.7)
- moved SW37 27.9 mm to (212.4, 126.4)
- moved C5 26.7 mm to (241.2, 163.5)
- moved C1 26.6 mm to (250.8, 156.2)
- moved C6 26.1 mm to (260.1, 162.2)
- moved C9 25.4 mm to (247.8, 167.0)
- moved J2 24.6 mm to (271.4, 151.3)
- moved SW65 23.5 mm to (319.3, 76.8)
- moved SW7 23.5 mm to (46.8, 95.9)
- moved SW27 21.3 mm to (131.6, 124.9)
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Connections:
- net +1V1 renamed /Right/1V1
- net /Left/col0L renamed /Left/matrixL/col0
- net /Left/col1L renamed /Left/matrixL/col1
- net /Left/col2L renamed /Left/matrixL/col2
- net /Left/col3L renamed /Left/matrixL/col3
- net /Left/col4L renamed /Left/matrixL/col4
- net /Left/col5L renamed /Left/matrixL/col5
- net /Left/col6L renamed /Left/matrixL/col6
- net /Left/row0L renamed /Left/matrixL/row0
- net /Left/row1L renamed /Left/matrixL/row1
- net /Left/row2L renamed /Left/matrixL/row2
- net /Left/row3L renamed /Left/matrixL/row3
- net /Left/row4L renamed /Left/matrixL/row4
- net /Right/col0L renamed /Right/matrixR/col0
- net /Right/col1L renamed /Right/matrixR/col1
- net /Right/col2L renamed /Right/matrixR/col2
- net /Right/col3L renamed /Right/matrixR/col3
- net /Right/col4L renamed /Right/matrixR/col4
- net /Right/col5L renamed /Right/matrixR/col5
- net /Right/col6L renamed /Right/matrixR/col6
- net /Right/row0L renamed /Right/matrixR/row0
- net /Right/row1L renamed /Right/matrixR/row1
- net /Right/row2L renamed /Right/matrixR/row2
- net /Right/row3L renamed /Right/matrixR/row3
- net /Right/row4L renamed /Right/matrixR/row4
- net VBUS renamed +5R
- C10 pad 1: +3V3 -> +3V3_L
- C11 pad 1: +3V3 -> +3V3_L
- C12 pad 1: +3V3 -> +3V3_L
- C13 pad 1: +3V3 -> +3V3_L
- C14 pad 1: +3V3 -> +3V3_L
- C15 pad 1: +3V3 -> +3V3_L
- C16 pad 1: +3V3 -> +3V3_L
- C4 pad 1: +3V3 -> +3V3_L
- C5 pad 1: +3V3 -> +3V3_L
- C9 pad 1: +3V3 -> +3V3_L
- R2 pad 1: +3V3 -> +3V3_L
- U1 pad 2: +3V3 -> +3V3_L
- U2 pad 8: +3V3 -> +3V3_L
- U3 pad 1: +3V3 -> +3V3_L
- U3 pad 10: +3V3 -> +3V3_L
- U3 pad 22: +3V3 -> +3V3_L
- U3 pad 26: /Right/RUN -> +3V3_L
- U3 pad 27: unconnected-(U3-Pad27) -> /Jack/TX_R
- U3 pad 28: unconnected-(U3-Pad28) -> /Jack/RX_R
- U3 pad 33: +3V3 -> +3V3_L
- U3 pad 42: +3V3 -> +3V3_L
- U3 pad 43: +3V3 -> +3V3_L
- U3 pad 44: +3V3 -> +3V3_L
- U3 pad 48: +3V3 -> +3V3_L
- U3 pad 49: +3V3 -> +3V3_L
- U3 pad 9: unconnected-(U3-Pad9) -> /Right/matrixR/col7
Routing:
- net (no net): track 0.32 -> 349.7 mm
- net /Left/matrixL/col6: track 88.4 -> 0.00 mm
- net /Left/matrixL/col4: track 65.6 -> 0.00 mm
- net /Right/matrixR/col1: track 64.6 -> 0.00 mm
- net /Right/matrixR/col3: track 64.6 -> 0.00 mm
- net /Left/matrixL/col0: track 41.5 -> 0.00 mm
- net /Right/matrixR/col6: track 24.7 -> 0.00 mm
