File: Plate left.kicad_sch (KiCad schematic)
At the start: 4 parts

Commit message: Left side gerbers generated
Parts:
- D68, D69: footprint LED_SMD:LED_0805_2012Metric -> arisu-split:LED_0805_2012Metric
Changed lines of the file:
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@@
     (property "Reference" "D68" (id 0) (at 90.4875 38.5912 0))
     (property "Value" "LED" (id 1) (at 90.4875 41.1281 0))
-    (property "Footprint" "LED_SMD:LED_0805_2012Metric" (id 2) (at 88.9 44.45 0)
+    (property "Footprint" "arisu-split:LED_0805_2012Metric" (id 2) (at 88.9 44.45 0)
       (effects (font (size 1.27 1.27)) hide)
     )
@@
     (property "Reference" "D69" (id 0) (at 90.4875 48.7512 0))
     (property "Value" "LED" (id 1) (at 90.4875 51.2881 0))
-    (property "Footprint" "LED_SMD:LED_0805_2012Metric" (id 2) (at 88.9 54.61 0)
+    (property "Footprint" "arisu-split:LED_0805_2012Metric" (id 2) (at 88.9 54.61 0)
       (effects (font (size 1.27 1.27)) hide)
     )
